File: MD試作/BLDC_Separated_ver1/Control/Control.kicad_pcb (KiCad board)
At the start: 4 copper layers, 35 x 35 mm, 98 parts, among them IC1 DCDC_MPM3620A, J1 Conn_01x14_Pin, J2 Conn_02x13_Odd_Even, J3 Conn_01x06_MountingPin, J4 Conn_01x06_MountingPin, Q1 BSS138, Q2 SSM3J332R, Q3 S8550, SW1 SW_SPST, SW3 SW_SPDT, SW4 SW_DIP_x04, U1 STM32G473CET6, U2 AZ1117CH-3.3, U3 MAX3485, U4 MAX3485, U5 Encoder_Magnetic_AS5047P, Y1 16MHz

Commit message: かんせい
Parts:
- added C26: 10uF, Capacitor_SMD:C_1206_3216Metric, F.Cu at (26.3, 16.5)
- added C27: 10uF, Capacitor_SMD:C_1206_3216Metric, F.Cu at (22.5, 17.9)
- L1: value 22uH -> 1uH; footprint MyLibrary:Inductor_CDPH4D19F -> Inductor_SMD:L_0603_1608Metric
- R15: value 10k -> 20k
- SW3: footprint MyLibrary:SW_Slide_DPDT_SSAJ120100 -> MyLibrary:SW_Slide_SPDT_SSAJ120100
- moved JP3 15.8 mm to (12.4, 27.2)
- moved L1 3.05 mm to (28.4, 13.7), turned to -90 degrees
- moved R14 1.80 mm to (32.4, 28.4)
- moved R24 1.13 mm to (8.68, 21.0)
- moved R13 0.75 mm to (32.5, 25.0)
- moved R16 0.35 mm to (17.6, 23.8)
- moved C24 0.15 mm to (16.6, 21.9)
- moved R22 0.12 mm to (11.5, 16.3)
- moved C7 0.12 mm to (9.81, 15.0), turned to 180 degrees
- moved R11 0.05 mm to (22.8, 21.3)
- turned C19 to -90 degrees
Connections:
- J2 pad 10: unconnected-(J2-Pin_10-Pad10) -> INC_L
- J2 pad 12: unconnected-(J2-Pin_12-Pad12) -> INA_L
- J2 pad 4: unconnected-(J2-Pin_4-Pad4) -> ENABLE
- J2 pad 6: unconnected-(J2-Pin_6-Pad6) -> nFAULT
- J2 pad 8: unconnected-(J2-Pin_8-Pad8) -> INB_L
- U1 pad 12: unconnected-(U1-PA4-Pad12) -> nFAULT
- U1 pad 2: unconnected-(U1-PC13-Pad2) -> INA_L
- U1 pad 3: unconnected-(U1-PC14-Pad3) -> INC_L
- U1 pad 34: unconnected-(U1-PA12-Pad34) -> ENABLE
- U1 pad 4: unconnected-(U1-PC15-Pad4) -> INB_L
Routing:
- net GND: track 226.5 -> 118.2 mm, vias 33 -> 217
- net +3.3V: track 13.4 -> 68.5 mm, vias 0 -> 55
- net INA_L: track 0.00 -> 34.3 mm, vias 0 -> 2
- net INC_L: track 0.00 -> 33.0 mm, vias 0 -> 1
- net ENABLE: track 0.00 -> 32.5 mm, vias 0 -> 2
- net INB_L: track 0.00 -> 30.3 mm, vias 0 -> 1
- net nFAULT: track 0.00 -> 26.0 mm, vias 0 -> 1
- net unconnected-(U1-PC13-Pad2): track 22.8 -> 0.00 mm, vias 2 -> 0
- net unconnected-(U1-PA12-Pad34): track 21.1 -> 0.00 mm, vias 2 -> 0
- net unconnected-(J2-Pin_10-Pad10): track 19.5 -> 0.00 mm
- net unconnected-(J2-Pin_8-Pad8): track 17.2 -> 0.00 mm
- net unconnected-(U1-PC14-Pad3): track 12.9 -> 0.00 mm, vias 1 -> 0
- net unconnected-(J2-Pin_6-Pad6): track 12.8 -> 0.00 mm
- net unconnected-(U1-PA4-Pad12): track 12.6 -> 0.00 mm, vias 1 -> 0
- net unconnected-(U1-PC15-Pad4): track 12.1 -> 0.00 mm, vias 1 -> 0
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- added copper zone on B.Cu, net +3.3V
- added copper zone on B.Cu, net +5V
- added copper zone on F.Cu, net +5V
- added copper zone on B.Cu, net /RS485/24V_IN
- added copper zone on F.Cu, net /RS485/24V_IN
- added copper zone on In1.Cu, net GND
Other:
- board text added: "JLCJLCJLCJLC"
- board text removed: "DIPスイッチ向き"
