File: MD試作/BLDC_Separated_ver1/Control/Power.kicad_sch (KiCad schematic)
At the start: 32 parts, among them IC1 DCDC_MPM3620A, Q3 BSS138, Q4 SSM3J332R, U4 AZ1117CH-3.3

Commit message: かんせい
Parts:
- added C26, C27: 10uF, Capacitor_SMD:C_1206_3216Metric, symbol Device:C
- L1: value 22uH -> 1uH; footprint MyLibrary:Inductor_CDPH4D19F -> Inductor_SMD:L_0603_1608Metric
- R31: value 10k -> 20k
Connections:
- net GND: now also C26.2, C27.2
- net VCC: now also C26.1, C27.1
Other:
- moved on the sheet: C14, C15, C20, C21
