File: MD試作/BLDC_Separated_ver1/Control/UI.kicad_sch (KiCad schematic)
At the start: 11 parts, among them SW3 SW_SPDT, SW4 SW_DIP_x04

Commit message: かんせい
Parts:
- SW3: footprint MyLibrary:SW_Slide_DPDT_SSAJ120100 -> MyLibrary:SW_Slide_SPDT_SSAJ120100
Changed lines of the file:
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@@
       (effects (font (size 1.27 1.27)) (justify left))
     )
-    (property "Footprint" "MyLibrary:SW_Slide_DPDT_SSAJ120100" (at 142.24 137.16 0)
+    (property "Footprint" "MyLibrary:SW_Slide_SPDT_SSAJ120100" (at 142.24 137.16 0)
       (effects (font (size 1.27 1.27)) hide)
     )

Commit message: ちょっと修正
Other:
- moved on the sheet: R31, R33, R6, R7, R8, SW3, SW4
