File: MD試作/BLDC_Separated_ver1/Control/RS485.kicad_sch (KiCad schematic)
At the start: 19 parts, among them J2 Conn_01x06_MountingPin, J3 Conn_01x06_MountingPin, Q1 S8550, U2 MAX3485, U3 MAX3485

Commit message: ちょっと修正
Connections:
- net RS485_A renamed RS485_RA
- net RS485_B renamed RS485_RB
- net RS485_X renamed RS485_TA
- net RS485_Y renamed RS485_TB
Other:
- note added: "MAX3485_Rx(3,4Pin)"
- note added: "MAX3485_Tx(5,6Pin)"
- note removed: "MAX3485_AB"
- note removed: "MAX3485_XY"
Changed lines of the file:
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@@
     (fill (type none))
+  )
+  (text "MAX3485_Tx(5,6Pin)" (at 73.66 99.06 0)
+    (effects (font (size 1.27 1.27)) (justify left bottom))
   )
   (text "RS485/Device" (at 73.66 30.48 0)
     (effects (font (size 2.54 2.54) (thickness 0.254) bold) (justify left bottom))
   )
-  (text "MAX3485_XY" (at 73.66 99.06 0)
+  (text "MAX3485_Rx(3,4Pin)" (at 73.66 38.1 0)
     (effects (font (size 1.27 1.27)) (justify left bottom))
   )
@@
     (effects (font (size 1.27 1.27)) (justify left bottom))
   )
-  (text "MAX3485_AB" (at 73.66 38.1 0)
-    (effects (font (size 1.27 1.27)) (justify left bottom))
-  )
   (text "24V_conn" (at 165.1 134.62 0)
     (effects (font (size 1.27 1.27)) (justify left bottom))
   )
-  (label "RS485_B" (at 182.88 58.42 180) (fields_autoplaced)
+  (label "RS485_RA" (at 147.32 58.42 0) (fields_autoplaced)
+    (effects (font (size 1.27 1.27) (thickness 0.254) bold) (justify left bottom))
+  )
+  (label "RS485_RA" (at 182.88 93.98 180) (fields_autoplaced)
     (effects (font (size 1.27 1.27) (thickness 0.254) bold) (justify right bottom))
   )
-  (label "RS485_X" (at 147.32 119.38 0) (fields_autoplaced)
+  (label "RS485_RA" (at 182.88 55.88 180) (fields_autoplaced)
+    (effects (font (size 1.27 1.27) (thickness 0.254) bold) (justify right bottom))
+  )
+  (label "RS485_TB" (at 182.88 101.6 180) (fields_autoplaced)
+    (effects (font (size 1.27 1.27) (thickness 0.254) bold) (justify right bottom))
+  )
+  (label "RS485_TB" (at 147.32 132.08 0) (fields_autoplaced)
     (effects (font (size 1.27 1.27) (thickness 0.254) bold) (justify left bottom))
   )
-  (label "RS485_B" (at 147.32 71.12 0) (fields_autoplaced)
-    (effects (font (size 1.27 1.27) (thickness 0.254) bold) (justify left bottom))
-  )
-  (label "RS485_Y" (at 182.88 101.6 180) (fields_autoplaced)
+  (label "RS485_TB" (at 182.88 63.5 180) (fields_autoplaced)
     (effects (font (size 1.27 1.27) (thickness 0.254) bold) (justify right bottom))
   )
-  (label "RS485_A" (at 182.88 93.98 180) (fields_autoplaced)
-    (effects (font (size 1.27 1.27) (thickness 0.254) bold) (justify right bottom))
-  )
-  (label "RS485_Y" (at 182.88 63.5 180) (fields_autoplaced)
+  (label "RS485_TA" (at 182.88 99.06 180) (fields_autoplaced)
     (effects (font (size 1.27 1.27) (thickness 0.254) bold) (justify right bottom))
   )
@@
     (effects (font (size 1.27 1.27) (thickness 0.254) bold) (justify right bottom))
   )
-  (label "RS485_A" (at 182.88 55.88 180) (fields_autoplaced)
+  (label "RS485_RB" (at 182.88 96.52 180) (fields_autoplaced)
+    (effects (font (size 1.27 1.27) (thickness 0.254) bold) (justify right bottom))
+  )
+  (label "RS485_RB" (at 182.88 58.42 180) (fields_autoplaced)
     (effects (font (size 1.27 1.27) (thickness 0.254) bold) (justify right bottom))
   )
@@
     (effects (font (size 1.27 1.27) (thickness 0.254) bold) (justify right bottom))
   )
-  (label "RS485_Y" (at 147.32 132.08 0) (fields_autoplaced)
+  (label "RS485_RB" (at 147.32 71.12 0) (fields_autoplaced)
     (effects (font (size 1.27 1.27) (thickness 0.254) bold) (justify left bottom))
   )
@@
     (effects (font (size 1.27 1.27) (thickness 0.254) bold) (justify left bottom))
   )
-  (label "RS485_A" (at 147.32 58.42 0) (fields_autoplaced)
+  (label "RS485_TA" (at 147.32 119.38 0) (fields_autoplaced)
     (effects (font (size 1.27 1.27) (thickness 0.254) bold) (justify left bottom))
-  )
-  (label "RS485_X" (at 182.88 60.96 180) (fields_autoplaced)
-    (effects (font (size 1.27 1.27) (thickness 0.254) bold) (justify right bottom))
   )
   (label "24V_IN" (at 177.8 142.24 180) (fields_autoplaced)
     (effects (font (size 1.27 1.27) (thickness 0.254) bold) (justify right bottom))
   )
-  (label "RS485_B" (at 182.88 96.52 180) (fields_autoplaced)
+  (label "RS485_TA" (at 182.88 60.96 180) (fields_autoplaced)
     (effects (font (size 1.27 1.27) (thickness 0.254) bold) (justify right bottom))
   )
-  (label "RS485_X" (at 182.88 99.06 180) (fields_autoplaced)
-    (effects (font (size 1.27 1.27) (thickness 0.254) bold) (justify right bottom))
-  )

Commit message: また修正
Other:
- note added: "RS485"
- note removed: "RS485/Device"
Changed lines of the file:
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@@
     (effects (font (size 1.27 1.27)) (justify left bottom))
   )
-  (text "RS485/Device" (at 73.66 30.48 0)
+  (text "RS485" (at 73.66 30.48 0)
     (effects (font (size 2.54 2.54) (thickness 0.254) bold) (justify left bottom))
   )
