File: MD試作/BLDC_Separated_ver1/MD/Power.kicad_sch (KiCad schematic)
At the start: 15 parts, among them J5 Conn_01x02_Pin, Q2 DI035P04PT, Q5 BSS138, Q6 DI035P04PT, SW4 SW_SPDT

Commit message: かんせい
Parts:
- added C2: 100uF, MyLibrary:Capacitor_Alum_Radial_5.0x11.0mm_Horizontal, symbol Device:C_Polarized
- added R4: 100k, Resistor_SMD:R_0402_1005Metric, symbol Device:R
- C17: footprint (none) -> MyLibrary:Capacitor_Alum_Radial_5.0x11.0mm_Horizontal
- R18: value 10k -> 47k
- R30: value 10k -> 20k
- SW4: footprint MyLibrary:SW_Slide_SPDT_SSSS820101 -> MyLibrary:SW_Slide_DPDT_SSSS820101
Connections:
- net GND: now also C2.2, R4.2
- net PowerSW: now also SW4.1 (A), R4.1; no longer R18.2, R19.1
- net S-S: now also R18.1; no longer SW4.2 (B)
- net VDD: now also C2.1
- new net: R18.2, R19.1, SW4.2 (B)
Other:
- moved on the sheet: R18, R19, SW4
