File: MD試作/BLDC_Separated_ver1/MD/MD.kicad_pcb (KiCad board)
At the start: 4 copper layers, 35 x 35 mm, 63 parts, among them J4 Conn_02x13_Odd_Even, J5 Conn_01x02_Pin, J6 Conn_01x03_Pin, Q10 TPN19008QM, Q11 TPN19008QM, Q12 TPN19008QM, Q2 DI035P04PT, Q5 BSS138, Q6 DI035P04PT, Q7 TPN19008QM, Q8 TPN19008QM, Q9 TPN19008QM, SW4 SW_SPDT, U6 Driver_FETGate_DRV8323S

Commit message: かんせい
Parts:
- added C1: 0.1uF, Capacitor_SMD:C_0402_1005Metric, B.Cu at (34.2, 16.7)
- added C17: 100uF, MyLibrary:Capacitor_Alum_Radial_5.0x11.0mm_Horizontal, B.Cu at (14.2, 0.10)
- added C2: 100uF, MyLibrary:Capacitor_Alum_Radial_5.0x11.0mm_Horizontal, B.Cu at (19.5, 0.10)
- added R3: 10k, Resistor_SMD:R_0402_1005Metric, B.Cu at (30.2, 26.0)
- added R4: 100k, Resistor_SMD:R_0402_1005Metric, B.Cu at (7.05, 10.0)
- D1: moved to F.Cu
- R18: value 10k -> 47k
- R30: value 10k -> 20k
- SW4: footprint MyLibrary:SW_Slide_SPDT_SSSS820101 -> MyLibrary:SW_Slide_DPDT_SSSS820101
- moved D5 32.6 mm to (19.6, 26.9), turned to -90 degrees
- moved R30 31.1 mm to (18.0, 26.5), turned to 90 degrees
- moved C14 23.6 mm to (1.39, 6.65)
- moved R28 16.4 mm to (6.52, 3.06), turned to -90 degrees
- moved R29 15.9 mm to (6.86, 4.62)
- moved Q5 15.8 mm to (6.08, 7.12), turned to 90 degrees
- moved R19 15.7 mm to (6.20, 12.6)
- moved R2 15.3 mm to (25.5, 12.8), turned to -135 degrees
- moved R18 13.3 mm to (3.35, 6.64)
- moved R24 10.5 mm to (7.60, 3.06), turned to -90 degrees
- moved R26 8.98 mm to (7.00, 1.42), turned to 0 degrees
- moved D1 6.15 mm to (34.0, 10.5), turned to -90 degrees
- moved R1 5.82 mm to (34.2, 14.7), turned to -90 degrees
- moved C24 5.56 mm to (21.8, 27.9), turned to -90 degrees
- moved C23 5.48 mm to (24.2, 27.9), turned to -90 degrees
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Connections:
- J4 pad 1: unconnected-(J4-Pin_1-Pad1) -> VDD
- J4 pad 10: unconnected-(J4-Pin_10-Pad10) -> INC_L
- J4 pad 11: unconnected-(J4-Pin_11-Pad11) -> MOSI1
- J4 pad 12: unconnected-(J4-Pin_12-Pad12) -> INA_L
- J4 pad 13: unconnected-(J4-Pin_13-Pad13) -> SCLK1
- J4 pad 14: unconnected-(J4-Pin_14-Pad14) -> CAL
- J4 pad 15: unconnected-(J4-Pin_15-Pad15) -> CS1_MD
- J4 pad 16: unconnected-(J4-Pin_16-Pad16) -> +3.3V
- J4 pad 17: unconnected-(J4-Pin_17-Pad17) -> INA_H
- J4 pad 18: unconnected-(J4-Pin_18-Pad18) -> GND
- J4 pad 19: unconnected-(J4-Pin_19-Pad19) -> INB_H
- J4 pad 2: unconnected-(J4-Pin_2-Pad2) -> VDD
- J4 pad 20: unconnected-(J4-Pin_20-Pad20) -> GND
- J4 pad 21: unconnected-(J4-Pin_21-Pad21) -> INC_H
- J4 pad 22: unconnected-(J4-Pin_22-Pad22) -> GND
- J4 pad 23: unconnected-(J4-Pin_23-Pad23) -> GND
- J4 pad 24: unconnected-(J4-Pin_24-Pad24) -> GND
- J4 pad 25: unconnected-(J4-Pin_25-Pad25) -> GND
- J4 pad 26: unconnected-(J4-Pin_26-Pad26) -> GND
- J4 pad 3: unconnected-(J4-Pin_3-Pad3) -> SOC
- J4 pad 4: unconnected-(J4-Pin_4-Pad4) -> ENABLE
- J4 pad 5: unconnected-(J4-Pin_5-Pad5) -> SOB
- J4 pad 6: unconnected-(J4-Pin_6-Pad6) -> nFAULT
- J4 pad 7: unconnected-(J4-Pin_7-Pad7) -> SOA
- J4 pad 8: unconnected-(J4-Pin_8-Pad8) -> INB_L
- J4 pad 9: unconnected-(J4-Pin_9-Pad9) -> MISO1
- R18 pad 1: Net-(SW4-A) -> /Power/S-S
- R18 pad 2: /Power/PowerSW -> Net-(SW4-B)
- R19 pad 1: /Power/PowerSW -> Net-(SW4-B)
- SW4 pad 1: Net-(SW4-A) -> /Power/PowerSW
- SW4 pad 2: /Power/S-S -> Net-(SW4-B)
Routing:
- net VDD: track 26.1 -> 88.1 mm, vias 0 -> 121
- net GND: track 25.8 -> 75.6 mm, vias 2 -> 217
- net /MotorDriver/Phase_U: track 0.00 -> 32.2 mm, vias 0 -> 53
- net +3.3V: track 1.60 -> 28.9 mm, vias 0 -> 2
- net Net-(Q6-G): track 0.00 -> 25.3 mm, vias 0 -> 2
- net CAL: track 0.00 -> 24.4 mm, vias 0 -> 3
- net Net-(Q2-G): track 0.00 -> 22.8 mm, vias 0 -> 2
- net nFAULT: track 0.00 -> 22.3 mm, vias 0 -> 1
- net /MotorDriver/Phase_V: track 0.00 -> 20.9 mm, vias 0 -> 47
- net INA_L: track 4.06 -> 24.0 mm, vias 1 -> 2
- net /Power/S-S: track 2.97 -> 22.5 mm, vias 0 -> 20
- net INB_L: track 4.42 -> 23.8 mm
- net /MotorDriver/Phase_W: track 0.00 -> 18.4 mm, vias 0 -> 51
- net ENABLE: track 0.00 -> 18.4 mm, vias 0 -> 2
- net INC_L: track 2.02 -> 19.4 mm, vias 0 -> 1
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- added copper zone on F.Cu, net /MotorDriver/BridgeA_S
- added copper zone on F.Cu, net /MotorDriver/BridgeB_S
- added copper zone on F.Cu, net /MotorDriver/BridgeC_S
- added copper zone on F.Cu, net /MotorDriver/Phase_U
- added copper zone on In1.Cu, net /MotorDriver/Phase_U
- added copper zone on In2.Cu, net /MotorDriver/Phase_U
- added copper zone on F.Cu, net /MotorDriver/Phase_V
- added copper zone on In1.Cu, net /MotorDriver/Phase_V
- added copper zone on In2.Cu, net /MotorDriver/Phase_V
- added copper zone on F.Cu, net /MotorDriver/Phase_W
- added copper zone on In1.Cu, net /MotorDriver/Phase_W
- added copper zone on In2.Cu, net /MotorDriver/Phase_W
- added copper zone on B.Cu, net /Power/S-S
- added copper zone on In1.Cu, net /Power/S-S
- added copper zone on In2.Cu, net /Power/S-S
- added copper zone on B.Cu, net GND
- added copper zone on In1.Cu, net GND
- added copper zone on In2.Cu, net GND
- added copper zone on B.Cu, net VDD
- added copper zone on In1.Cu, net VDD
- added copper zone on In2.Cu, net VDD
Other:
- board text added: "Designed by @cat_nekonekone"
- board text added: "JLCJLCJLCJLC"
- board text added: "U"
- board text added: "V"
- board text added: "W"
- board text added: "燈"

Commit message: 発注後修正1
Routing:
- net GND: vias 217 -> 212
Changed lines of the file:
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@@
   (via (at 29.303917 28.013254) (size 0.45) (drill 0.3) (layers "F.Cu" "B.Cu") (free) (net 4))
   (via (at 22.75 34) (size 0.45) (drill 0.3) (layers "F.Cu" "B.Cu") (free) (net 4))
-  (via (at 18.100705 6.895796) (size 0.45) (drill 0.3) (layers "F.Cu" "B.Cu") (free) (net 4))
+  (via (at 17.85 6.95) (size 0.45) (drill 0.3) (layers "F.Cu" "B.Cu") (free) (net 4))
   (via (at 25.468466 18.011122) (size 0.45) (drill 0.3) (layers "F.Cu" "B.Cu") (net 4))
   (via (at 7.866903 11.731696) (size 0.45) (drill 0.3) (layers "F.Cu" "B.Cu") (free) (net 4))
@@
   (via (at 26.698716 3.51793) (size 0.45) (drill 0.3) (layers "F.Cu" "B.Cu") (free) (net 4))
   (via (at 29.982009 10.367076) (size 0.45) (drill 0.3) (layers "F.Cu" "B.Cu") (free) (net 4))
-  (via (at 23.75 5.25) (size 0.45) (drill 0.3) (layers "F.Cu" "B.Cu") (free) (net 4))
   (via (at 28.27476 24.821045) (size 0.45) (drill 0.3) (layers "F.Cu" "B.Cu") (free) (net 4))
   (via (at 18.733451 7.810217) (size 0.45) (drill 0.3) (layers "F.Cu" "B.Cu") (free) (net 4))
@@
   (via (at 1.8 33.6) (size 0.45) (drill 0.3) (layers "F.Cu" "B.Cu") (free) (net 4))
   (via (at 8.25 2) (size 0.45) (drill 0.3) (layers "F.Cu" "B.Cu") (free) (net 4))
-  (via (at 21.015422 5.729515) (size 0.45) (drill 0.3) (layers "F.Cu" "B.Cu") (free) (net 4))
   (via (at 26.959631 29.371422) (size 0.45) (drill 0.3) (layers "F.Cu" "B.Cu") (net 4))
   (via (at 33.25 33.5) (size 0.45) (drill 0.3) (layers "F.Cu" "B.Cu") (free) (net 4))
@@
   (via (at 29.173765 21.402366) (size 0.45) (drill 0.3) (layers "F.Cu" "B.Cu") (free) (net 4))
   (via (at 28.266181 21.415332) (size 0.45) (drill 0.3) (layers "F.Cu" "B.Cu") (free) (net 4))
-  (via (at 22.238945 6.912995) (size 0.45) (drill 0.3) (layers "F.Cu" "B.Cu") (free) (net 4))
   (via (at 28.082808 10.323724) (size 0.45) (drill 0.3) (layers "F.Cu" "B.Cu") (net 4))
   (via (at 29.946357 12.960821) (size 0.45) (drill 0.3) (layers "F.Cu" "B.Cu") (free) (net 4))
-  (via (at 20.75 2.25) (size 0.45) (drill 0.3) (layers "F.Cu" "B.Cu") (free) (net 4))
+  (via (at 20.9 2.05) (size 0.45) (drill 0.3) (layers "F.Cu" "B.Cu") (free) (net 4))
   (via (at 24.962349 28.116426) (size 0.45) (drill 0.3) (layers "F.Cu" "B.Cu") (free) (net 4))
   (via (at 7.595912 5.543687) (size 0.45) (drill 0.3) (layers "F.Cu" "B.Cu") (free) (net 4))
@@
   (via (at 28.668345 27.424521) (size 0.45) (drill 0.3) (layers "F.Cu" "B.Cu") (free) (net 4))
   (via (at 30 34) (size 0.45) (drill 0.3) (layers "F.Cu" "B.Cu") (free) (net 4))
-  (via (at 21.099956 6.899647) (size 0.45) (drill 0.3) (layers "F.Cu" "B.Cu") (free) (net 4))
   (via (at 22.990265 18.090221) (size 0.45) (drill 0.3) (layers "F.Cu" "B.Cu") (net 4))
   (via (at 19.204805 15.468521) (size 0.45) (drill 0.3) (layers "F.Cu" "B.Cu") (free) (net 4))
@@
   (via (at 2 8.8) (size 0.45) (drill 0.3) (layers "F.Cu" "B.Cu") (free) (net 4))
   (via (at 32 29.2) (size 0.45) (drill 0.3) (layers "F.Cu" "B.Cu") (free) (net 4))
-  (via (at 17.25 6.25) (size 0.45) (drill 0.3) (layers "F.Cu" "B.Cu") (free) (net 4))
+  (via (at 17 6.35) (size 0.45) (drill 0.3) (layers "F.Cu" "B.Cu") (free) (net 4))
   (via (at 22.972721 32.233427) (size 0.45) (drill 0.3) (layers "F.Cu" "B.Cu") (free) (net 4))
   (via (at 29.398304 24.244577) (size 0.45) (drill 0.3) (layers "F.Cu" "B.Cu") (free) (net 4))
@@
   (via (at 29.935007 11.561298) (size 0.45) (drill 0.3) (layers "F.Cu" "B.Cu") (free) (net 4))
   (via (at 27.005545 31.70541) (size 0.45) (drill 0.3) (layers "F.Cu" "B.Cu") (net 4))
-  (via (at 24.114795 8.176756) (size 0.45) (drill 0.3) (layers "F.Cu" "B.Cu") (free) (net 4))
+  (via (at 23.85 8.5) (size 0.45) (drill 0.3) (layers "F.Cu" "B.Cu") (free) (net 4))
   (via (at 26.618399 20.085403) (size 0.45) (drill 0.3) (layers "F.Cu" "B.Cu") (free) (net 4))
-  (via (at 19.681317 2.249359) (size 0.45) (drill 0.3) (layers "F.Cu" "B.Cu") (free) (net 4))
-  (via (at 18.5 2.25) (size 0.45) (drill 0.3) (layers "F.Cu" "B.Cu") (free) (net 4))
+  (via (at 19.8 2.05) (size 0.45) (drill 0.3) (layers "F.Cu" "B.Cu") (free) (net 4))
+  (via (at 18.65 2.05) (size 0.45) (drill 0.3) (layers "F.Cu" "B.Cu") (free) (net 4))
   (via (at 10.8 33.4) (size 0.45) (drill 0.3) (layers "F.Cu" "B.Cu") (free) (net 4))
   (via (at 28.033289 9.024165) (size 0.45) (drill 0.3) (layers "F.Cu" "B.Cu") (net 4))
@@
   (via (at 25.491054 29.998255) (size 0.45) (drill 0.3) (layers "F.Cu" "B.Cu") (free) (net 4))
   (via (at 26.885587 10.524244) (size 0.45) (drill 0.3) (layers "F.Cu" "B.Cu") (net 4))
-  (via (at 23.562945 3.772711) (size 0.45) (drill 0.3) (layers "F.Cu" "B.Cu") (free) (net 4))
+  (via (at 23.75 3.55) (size 0.45) (drill 0.3) (layers "F.Cu" "B.Cu") (free) (net 4))
   (via (at 28.269516 22.210886) (size 0.45) (drill 0.3) (layers "F.Cu" "B.Cu") (free) (net 4))
   (via (at 2 4.75) (size 0.45) (drill 0.3) (layers "F.Cu" "B.Cu") (free) (net 4))
@@
   (via (at 27.510605 32.256384) (size 0.45) (drill 0.3) (layers "F.Cu" "B.Cu") (net 4))
   (via (at 27.75 4) (size 0.45) (drill 0.3) (layers "F.Cu" "B.Cu") (free) (net 4))
-  (via (at 22.083254 2.665392) (size 0.45) (drill 0.3) (layers "F.Cu" "B.Cu") (free) (net 4))
+  (via (at 22.2 2.25) (size 0.45) (drill 0.3) (layers "F.Cu" "B.Cu") (free) (net 4))
   (via (at 29.75 1.75) (size 0.45) (drill 0.3) (layers "F.Cu" "B.Cu") (free) (net 4))
   (via (at 30.75 1) (size 0.45) (drill 0.3) (layers "F.Cu" "B.Cu") (free) (net 4))
@@
   (via (at 24.462839 28.770109) (size 0.45) (drill 0.3) (layers "F.Cu" "B.Cu") (net 4))
   (via (at 28.070936 5.728687) (size 0.45) (drill 0.3) (layers "F.Cu" "B.Cu") (free) (net 4))
-  (via (at 19 6.25) (size 0.45) (drill 0.3) (layers "F.Cu" "B.Cu") (free) (net 4))
+  (via (at 18.75 6.95) (size 0.45) (drill 0.3) (layers "F.Cu" "B.Cu") (free) (net 4))
   (via (at 23.048628 20.491082) (size 0.45) (drill 0.3) (layers "F.Cu" "B.Cu") (net 4))
   (via (at 28.28779 23.148385) (size 0.45) (drill 0.3) (layers "F.Cu" "B.Cu") (free) (net 4))
@@
   (via (at 24.380766 32.317603) (size 0.45) (drill 0.3) (layers "F.Cu" "B.Cu") (free) (net 4))
   (via (at 29.5 5.75) (size 0.45) (drill 0.3) (layers "F.Cu" "B.Cu") (free) (net 4))
-  (via (at 22.25 3.75) (size 0.45) (drill 0.3) (layers "F.Cu" "B.Cu") (free) (net 4))
   (via (at 26.612896 17.004243) (size 0.45) (drill 0.3) (layers "F.Cu" "B.Cu") (free) (net 4))
   (via (at 28.75808 23.568373) (size 0.45) (drill 0.3) (layers "F.Cu" "B.Cu") (free) (net 4))
@@
   )
   (zone (net 25) (net_name "/Power/24VBAT") (layer "F.Cu") (hatch edge 0.5)
+    (priority 1)
     (connect_pads yes (clearance 0.2))
     (min_thickness 0.25) (filled_areas_thickness no)
